Commit message: feat: 改差速为阿克曼转向底盘
- genbot.urdf.xacro: 前轮转向节(steering_link)+转向关节(绕Z轴)+滚动关节(绕Y轴)，后轮仅驱动
- genbot.gazebo.xacro: DiffDrive驱动后轮 + JointPositionController控制前轮转向
- 新增 genbot_control 包，ackermann_steering_node.py 计算阿克曼转角
- gazebo.launch.py: 加入阿克曼节点和转向话题桥接

File: software/genbot_description/urdf/genbot.gazebo.xacro (robot description, xacro)
@@ -3,12 +3,11 @@
   <!--
    ============================================================
-    Gazebo Harmonic (gz-sim 8) 插件配置
+    GenBot Ackermann — Gazebo Harmonic (gz-sim 8) 插件配置
    ============================================================
-   Gazebo Harmonic 使用 <gz::sim::systems::...> 命名空间
-   不再使用旧版 <gazebo> 标签中的 libgazebo_ros_*.so
-   通过 ros_gz_bridge 桥接 ROS2 ↔ Gazebo 通信
+   后轮: DiffDrive（速度控制）
+   前轮: JointPositionController（位置控制，阿克曼转角）
    ============================================================
   -->
-  <!-- 底盘物理参数 -->
+  <!-- 底盘物理 -->
   <gazebo reference="base_link">
     <material>Gazebo/Grey</material>
@@ -21,6 +20,6 @@
     <friction2>0.5</friction2>
   </gazebo>
-  <!-- 驱动轮物理参数 -->
-  <gazebo reference="left_wheel">
+  <!-- 后轮驱动 — 高摩擦 -->
+  <gazebo reference="rear_left_wheel">
     <mu1>1.0</mu1>
     <mu2>1.0</mu2>
@@ -29,5 +28,5 @@
     <material>Gazebo/Black</material>
   </gazebo>
-  <gazebo reference="right_wheel">
+  <gazebo reference="rear_right_wheel">
     <mu1>1.0</mu1>
     <mu2>1.0</mu2>
@@ -36,19 +35,33 @@
     <material>Gazebo/Black</material>
   </gazebo>
-  <!-- 万向轮：低摩擦 -->
-  <gazebo reference="caster_front_left_wheel">
-    <mu1>0.01</mu1>
-    <mu2>0.01</mu2>
+  <!-- 前轮转向节 — 中等摩擦 -->
+  <gazebo reference="front_left_steering_link">
+    <mu1>0.3</mu1>
+    <mu2>0.3</mu2>
   </gazebo>
-  <gazebo reference="caster_front_right_wheel">
-    <mu1>0.01</mu1>
-    <mu2>0.01</mu2>
+  <gazebo reference="front_right_steering_link">
+    <mu1>0.3</mu1>
+    <mu2>0.3</mu2>
   </gazebo>
-  <!-- 差速驱动系统（gz-sim原生插件） -->
+  <!-- 前轮 — 低摩擦（转向轮需要低侧向摩擦） -->
+  <gazebo reference="front_left_wheel">
+    <mu1>0.3</mu1>
+    <mu2>0.3</mu2>
+    <material>Gazebo/Black</material>
+  </gazebo>
+  <gazebo reference="front_right_wheel">
+    <mu1>0.3</mu1>
+    <mu2>0.3</mu2>
+    <material>Gazebo/Black</material>
+  </gazebo>
+  <!-- ============================================================ -->
+  <!--  后轮差速驱动（DiffDrive）                                    -->
+  <!--  订阅 /cmd_vel 中的 linear.x 速度                            -->
+  <!-- ============================================================ -->
   <gazebo>
     <plugin filename="libgz-sim-diff-drive-system.so"
             name="gz::sim::systems::DiffDrive">
-      <left_joint>left_wheel_joint</left_joint>
-      <right_joint>right_wheel_joint</right_joint>
+      <left_joint>rear_left_wheel_joint</left_joint>
+      <right_joint>rear_right_wheel_joint</right_joint>
       <wheel_separation>${wheel_track}</wheel_separation>
       <wheel_radius>${wheel_radius}</wheel_radius>
@@ -64,5 +77,36 @@
     </plugin>
   </gazebo>
-  <!-- LiDAR 传感器 -->
+  <!-- ============================================================ -->
+  <!--  前轮转向控制（JointPositionController）                     -->
+  <!--  通过 /cmd_steer_left 和 /cmd_steer_right 控制转向角度       -->
+  <!--  阿克曼转角由外部节点计算后发布                               -->
+  <!-- ============================================================ -->
+  <gazebo>
+    <plugin filename="libgz-sim-joint-position-controller-system.so"
+            name="gz::sim::systems::JointPositionController">
+      <joint_name>front_left_steering_joint</joint_name>
+      <topic>/cmd_steer_left</topic>
+      <use_cmd_composition>true</use_cmd_composition>
+      <publish_cmd>true</publish_cmd>
+      <publish_state>true</publish_state>
+      <publish_pose>true</publish_pose>
+      <publish_wrench>false</publish_wrench>
+    </plugin>
+  </gazebo>
+  <gazebo>
+    <plugin filename="libgz-sim-joint-position-controller-system.so"
+            name="gz::sim::systems::JointPositionController">
+      <joint_name>front_right_steering_joint</joint_name>
+      <topic>/cmd_steer_right</topic>
+      <use_cmd_composition>true</use_cmd_composition>
+      <publish_cmd>true</publish_cmd>
+      <publish_state>true</publish_state>
+      <publish_pose>true</publish_pose>
+      <publish_wrench>false</publish_wrench>
+    </plugin>
+  </gazebo>
+  <!-- ============================================================ -->
+  <!--  LiDAR                                                       -->
+  <!-- ============================================================ -->
   <gazebo reference="lidar_link">
     <sensor name="lidar" type="gpu_lidar">
@@ -70,11 +114,17 @@
       <update_rate>10</update_rate>
       <lidar>
-        <scan_count>1</scan_count>
-        <scan_angle_start>0.0</scan_angle_start>
-        <scan_angle_end>6.283185</scan_angle_end>
-        <scan_samples>360</scan_samples>
-        <range_min>0.15</range_min>
-        <range_max>12.0</range_max>
-        <range_resolution>0.015</range_resolution>
+        <scan>
+          <horizontal>
+            <samples>360</samples>
+            <resolution>1.0</resolution>
+            <min_angle>0.0</min_angle>
+            <max_angle>6.283185</max_angle>
+          </horizontal>
+        </scan>
+        <range>
+          <min>0.15</min>
+          <max>12.0</max>
+          <resolution>0.015</resolution>
+        </range>
       </lidar>
       <noise>
@@ -87,5 +137,7 @@
     </sensor>
   </gazebo>
-  <!-- RGB 相机 -->
+  <!-- ============================================================ -->
+  <!--  RGB 相机 + 深度相机                                         -->
+  <!-- ============================================================ -->
   <gazebo reference="camera_link">
     <sensor name="rgb_camera" type="camera">
@@ -107,5 +159,4 @@
       <visualize>true</visualize>
     </sensor>
-    <!-- 深度相机 -->
     <sensor name="depth_camera" type="depth_camera">
       <topic>/camera/depth/image_raw</topic>
@@ -127,5 +178,7 @@
     </sensor>
   </gazebo>
-  <!-- IMU -->
+  <!-- ============================================================ -->
+  <!--  IMU                                                        -->
+  <!-- ============================================================ -->
   <gazebo reference="imu_link">
     <sensor name="imu" type="imu">

File: software/genbot_description/urdf/genbot.urdf.xacro (robot description, xacro)
@@ -3,14 +3,13 @@
   <!--
    ============================================================
-    GenBot 4WD — 4轮差速通用机器人开发平台
+    GenBot Ackermann — 阿克曼转向通用机器人开发平台
    ============================================================
-   底盘: 350mm x 280mm
+   底盘: 400mm x 280mm
+   转向: 前轮阿克曼转向（左右转角不同）
    驱动: 后轮JGA25-371直流有刷编码电机
-   从动: 前工业万向轮
    传感器: RPLIDAR A1 (顶) + Realsense D435 (前) + MPU6050 (内)
    仿真: Gazebo Harmonic (gz-sim 8)
    ============================================================
   -->
-  <!-- 颜色定义 -->
   <material name="ChassisGray">
     <color rgba="0.25 0.25 0.28 1.0"/>
@@ -19,5 +18,5 @@
     <color rgba="0.08 0.08 0.08 1.0"/>
   </material>
-  <material name="CasterSilver">
+  <material name="UprightSilver">
     <color rgba="0.70 0.70 0.72 1.0"/>
   </material>
@@ -32,14 +31,12 @@
   </material>
   <!-- ========== 机器人参数 ========== -->
-  <xacro:property name="chassis_length"  value="0.350"/>
-  <xacro:property name="chassis_width"   value="0.280"/>
-  <xacro:property name="chassis_height"  value="0.080"/>
-  <xacro:property name="clearance"       value="0.050"/>
-  <xacro:property name="wheel_radius"    value="0.050"/>
-  <xacro:property name="wheel_width"     value="0.035"/>
-  <xacro:property name="wheel_track"     value="0.240"/>
-  <xacro:property name="wheel_base"      value="0.220"/>
-  <xacro:property name="caster_radius"   value="0.020"/>
-  <xacro:property name="caster_arm"      value="0.025"/>
+  <xacro:property name="wheel_base"    value="0.300"/>
+  <xacro:property name="wheel_track"   value="0.240"/>
+  <xacro:property name="chassis_length" value="0.400"/>
+  <xacro:property name="chassis_width"  value="0.280"/>
+  <xacro:property name="chassis_height" value="0.080"/>
+  <xacro:property name="clearance"      value="0.050"/>
+  <xacro:property name="wheel_radius"   value="0.050"/>
+  <xacro:property name="wheel_width"    value="0.035"/>
   <!-- ========== 惯性宏 ========== -->
   <xacro:macro name="inertia_box" params="mass x y z">
@@ -61,14 +58,5 @@
     </inertial>
   </xacro:macro>
-  <xacro:macro name="inertia_sphere" params="mass r">
-    <inertial>
-      <mass value="${mass}"/>
-      <inertia ixx="${0.4*mass*r*r}"
-               iyy="${0.4*mass*r*r}"
-               izz="${0.4*mass*r*r}"
-               ixy="0" iyz="0" ixz="0"/>
-    </inertial>
-  </xacro:macro>
-  <!-- ========== base_footprint（地面投影）========== -->
+  <!-- ========== base_footprint ========== -->
   <link name="base_footprint"/>
   <!-- ========== 底盘 ========== -->
@@ -90,20 +78,108 @@
     <origin xyz="0 0 ${clearance + chassis_height/2}" rpy="0 0 0"/>
   </joint>
-  <!-- ========== 后轮 — 驱动轮（左）========== -->
-  <link name="left_wheel">
-    <visual>
-      <origin xyz="0 0 0" rpy="${pi/2} 0 0"/>
-      <geometry><cylinder radius="${wheel_radius}" length="${wheel_width}"/></geometry>
-      <material name="WheelBlack"/>
-    </visual>
-    <collision>
-      <origin xyz="0 0 0" rpy="${pi/2} 0 0"/>
-      <geometry><cylinder radius="${wheel_radius}" length="${wheel_width}"/></geometry>
-    </collision>
-    <xacro:inertia_cyl mass="0.3" r="${wheel_radius}" l="${wheel_width}"/>
-  </link>
-  <joint name="left_wheel_joint" type="continuous">
-    <parent link="base_link"/>
-    <child link="left_wheel"/>
+  <!-- ================================================================ -->
+  <!--  前轮 — 左（转向节 + 转向关节 + 轮子 + 滚动关节）                -->
+  <!-- ================================================================ -->
+  <link name="front_left_steering_link">
+    <visual>
+      <origin xyz="0 0 0" rpy="0 0 0"/>
+      <geometry><box size="0.030 0.030 0.080"/></geometry>
+      <material name="UprightSilver"/>
+    </visual>
+    <collision>
+      <origin xyz="0 0 0" rpy="0 0 0"/>
+      <geometry><box size="0.030 0.030 0.080"/></geometry>
+    </collision>
+    <xacro:inertia_box mass="0.15" x="0.03" y="0.03" z="0.08"/>
+  </link>
+  <joint name="front_left_steering_joint" type="revolute">
+    <parent link="base_link"/>
+    <child link="front_left_steering_link"/>
+    <origin xyz="${wheel_base/2} ${wheel_track/2} ${-chassis_height/2}" rpy="0 0 0"/>
+    <axis xyz="0 0 1"/>
+    <limit effort="10.0" velocity="3.0" lower="-0.6" upper="0.6"/>
+    <dynamics damping="0.05" friction="0.01"/>
+  </joint>
+  <link name="front_left_wheel">
+    <visual>
+      <origin xyz="0 0 0" rpy="${pi/2} 0 0"/>
+      <geometry><cylinder radius="${wheel_radius}" length="${wheel_width}"/></geometry>
+      <material name="WheelBlack"/>
+    </visual>
+    <collision>
+      <origin xyz="0 0 0" rpy="${pi/2} 0 0"/>
+      <geometry><cylinder radius="${wheel_radius}" length="${wheel_width}"/></geometry>
+    </collision>
+    <xacro:inertia_cyl mass="0.3" r="${wheel_radius}" l="${wheel_width}"/>
+  </link>
+  <joint name="front_left_wheel_joint" type="continuous">
+    <parent link="front_left_steering_link"/>
+    <child link="front_left_wheel"/>
+    <origin xyz="0 0 -0.045" rpy="0 0 0"/>
+    <axis xyz="0 1 0"/>
+    <limit effort="0.5" velocity="10.0"/>
+    <dynamics damping="0.01" friction="0.01"/>
+  </joint>
+  <!-- ================================================================ -->
+  <!--  前轮 — 右                                                      -->
+  <!-- ================================================================ -->
+  <link name="front_right_steering_link">
+    <visual>
+      <origin xyz="0 0 0" rpy="0 0 0"/>
+      <geometry><box size="0.030 0.030 0.080"/></geometry>
+      <material name="UprightSilver"/>
+    </visual>
+    <collision>
+      <origin xyz="0 0 0" rpy="0 0 0"/>
+      <geometry><box size="0.030 0.030 0.080"/></geometry>
+    </collision>
+    <xacro:inertia_box mass="0.15" x="0.03" y="0.03" z="0.08"/>
+  </link>
+  <joint name="front_right_steering_joint" type="revolute">
+    <parent link="base_link"/>
+    <child link="front_right_steering_link"/>
+    <origin xyz="${wheel_base/2} ${-wheel_track/2} ${-chassis_height/2}" rpy="0 0 0"/>
+    <axis xyz="0 0 1"/>
+    <limit effort="10.0" velocity="3.0" lower="-0.6" upper="0.6"/>
+    <dynamics damping="0.05" friction="0.01"/>
+  </joint>
+  <link name="front_right_wheel">
+    <visual>
+      <origin xyz="0 0 0" rpy="${pi/2} 0 0"/>
+      <geometry><cylinder radius="${wheel_radius}" length="${wheel_width}"/></geometry>
+      <material name="WheelBlack"/>
+    </visual>
+    <collision>
+      <origin xyz="0 0 0" rpy="${pi/2} 0 0"/>
+      <geometry><cylinder radius="${wheel_radius}" length="${wheel_width}"/></geometry>
+    </collision>
+    <xacro:inertia_cyl mass="0.3" r="${wheel_radius}" l="${wheel_width}"/>
+  </link>
+  <joint name="front_right_wheel_joint" type="continuous">
+    <parent link="front_right_steering_link"/>
+    <child link="front_right_wheel"/>
+    <origin xyz="0 0 -0.045" rpy="0 0 0"/>
+    <axis xyz="0 1 0"/>
+    <limit effort="0.5" velocity="10.0"/>
+    <dynamics damping="0.01" friction="0.01"/>
+  </joint>
+  <!-- ================================================================ -->
+  <!--  后轮 — 左（仅驱动，不转向）                                    -->
+  <!-- ================================================================ -->
+  <link name="rear_left_wheel">
+    <visual>
+      <origin xyz="0 0 0" rpy="${pi/2} 0 0"/>
+      <geometry><cylinder radius="${wheel_radius}" length="${wheel_width}"/></geometry>
+      <material name="WheelBlack"/>
+    </visual>
+    <collision>
+      <origin xyz="0 0 0" rpy="${pi/2} 0 0"/>
+      <geometry><cylinder radius="${wheel_radius}" length="${wheel_width}"/></geometry>
+    </collision>
+    <xacro:inertia_cyl mass="0.3" r="${wheel_radius}" l="${wheel_width}"/>
+  </link>
+  <joint name="rear_left_wheel_joint" type="continuous">
+    <parent link="base_link"/>
+    <child link="rear_left_wheel"/>
     <origin xyz="${-wheel_base/2} ${wheel_track/2} ${-chassis_height/2}" rpy="0 0 0"/>
     <axis xyz="0 1 0"/>
@@ -111,102 +187,26 @@
     <dynamics damping="0.01" friction="0.01"/>
   </joint>
-  <!-- ========== 后轮 — 驱动轮（右）========== -->
-  <link name="right_wheel">
-    <visual>
-      <origin xyz="0 0 0" rpy="${pi/2} 0 0"/>
-      <geometry><cylinder radius="${wheel_radius}" length="${wheel_width}"/></geometry>
-      <material name="WheelBlack"/>
-    </visual>
-    <collision>
-      <origin xyz="0 0 0" rpy="${pi/2} 0 0"/>
-      <geometry><cylinder radius="${wheel_radius}" length="${wheel_width}"/></geometry>
-    </collision>
-    <xacro:inertia_cyl mass="0.3" r="${wheel_radius}" l="${wheel_width}"/>
-  </link>
-  <joint name="right_wheel_joint" type="continuous">
-    <parent link="base_link"/>
-    <child link="right_wheel"/>
+  <!-- ================================================================ -->
+  <!--  后轮 — 右                                                      -->
+  <!-- ================================================================ -->
+  <link name="rear_right_wheel">
+    <visual>
+      <origin xyz="0 0 0" rpy="${pi/2} 0 0"/>
+      <geometry><cylinder radius="${wheel_radius}" length="${wheel_width}"/></geometry>
+      <material name="WheelBlack"/>
+    </visual>
+    <collision>
+      <origin xyz="0 0 0" rpy="${pi/2} 0 0"/>
+      <geometry><cylinder radius="${wheel_radius}" length="${wheel_width}"/></geometry>
+    </collision>
+    <xacro:inertia_cyl mass="0.3" r="${wheel_radius}" l="${wheel_width}"/>
+  </link>
+  <joint name="rear_right_wheel_joint" type="continuous">
+    <parent link="base_link"/>
+    <child link="rear_right_wheel"/>
     <origin xyz="${-wheel_base/2} ${-wheel_track/2} ${-chassis_height/2}" rpy="0 0 0"/>
     <axis xyz="0 1 0"/>
     <limit effort="0.5" velocity="10.0"/>
     <dynamics damping="0.01" friction="0.01"/>
-  </joint>
-  <!-- ========== 前万向轮 — 左 ========== -->
-  <link name="caster_front_left_fork">
-    <visual>
-      <origin xyz="0 0 ${-caster_arm/2}" rpy="0 0 0"/>
-      <geometry><cylinder radius="0.008" length="${caster_arm}"/></geometry>
-      <material name="CasterSilver"/>
-    </visual>
-    <collision>
-      <origin xyz="0 0 ${-caster_arm/2}" rpy="0 0 0"/>
-      <geometry><cylinder radius="0.008" length="${caster_arm}"/></geometry>
-    </collision>
-    <xacro:inertia_cyl mass="0.03" r="0.008" l="${caster_arm}"/>
-  </link>
-  <joint name="caster_front_left_fork_joint" type="continuous">
-    <parent link="base_link"/>
-    <child link="caster_front_left_fork"/>
-    <origin xyz="${chassis_length/2 - 0.030} ${0.100} ${-chassis_height/2}" rpy="0 0 0"/>
-    <axis xyz="0 0 1"/>
-    <dynamics damping="0.001" friction="0.001"/>
-  </joint>
-  <link name="caster_front_left_wheel">
-    <visual>
-      <origin xyz="0 0 ${-caster_arm}" rpy="0 0 0"/>
-      <geometry><sphere radius="${caster_radius}"/></geometry>
-      <material name="WheelBlack"/>
-    </visual>
-    <collision>
-      <origin xyz="0 0 ${-caster_arm}" rpy="0 0 0"/>
-      <geometry><sphere radius="${caster_radius}"/></geometry>
-    </collision>
-    <xacro:inertia_sphere mass="0.05" r="${caster_radius}"/>
-  </link>
-  <joint name="caster_front_left_wheel_joint" type="continuous">
-    <parent link="caster_front_left_fork"/>
-    <child link="caster_front_left_wheel"/>
-    <origin xyz="0 0 ${-caster_arm}" rpy="0 0 0"/>
-    <axis xyz="0 1 0"/>
-    <dynamics damping="0.001" friction="0.001"/>
-  </joint>
-  <!-- ========== 前万向轮 — 右 ========== -->
-  <link name="caster_front_right_fork">
-    <visual>
-      <origin xyz="0 0 ${-caster_arm/2}" rpy="0 0 0"/>
-      <geometry><cylinder radius="0.008" length="${caster_arm}"/></geometry>
-      <material name="CasterSilver"/>
-    </visual>
-    <collision>
-      <origin xyz="0 0 ${-caster_arm/2}" rpy="0 0 0"/>
-      <geometry><cylinder radius="0.008" length="${caster_arm}"/></geometry>
-    </collision>
-    <xacro:inertia_cyl mass="0.03" r="0.008" l="${caster_arm}"/>
-  </link>
-  <joint name="caster_front_right_fork_joint" type="continuous">
-    <parent link="base_link"/>
-    <child link="caster_front_right_fork"/>
-    <origin xyz="${chassis_length/2 - 0.030} ${-0.100} ${-chassis_height/2}" rpy="0 0 0"/>
-    <axis xyz="0 0 1"/>
-    <dynamics damping="0.001" friction="0.001"/>
-  </joint>
-  <link name="caster_front_right_wheel">
-    <visual>
-      <origin xyz="0 0 ${-caster_arm}" rpy="0 0 0"/>
-      <geometry><sphere radius="${caster_radius}"/></geometry>
-      <material name="WheelBlack"/>
-    </visual>
-    <collision>
-      <origin xyz="0 0 ${-caster_arm}" rpy="0 0 0"/>
-      <geometry><sphere radius="${caster_radius}"/></geometry>
-    </collision>
-    <xacro:inertia_sphere mass="0.05" r="${caster_radius}"/>
-  </link>
-  <joint name="caster_front_right_wheel_joint" type="continuous">
-    <parent link="caster_front_right_fork"/>
-    <child link="caster_front_right_wheel"/>
-    <origin xyz="0 0 ${-caster_arm}" rpy="0 0 0"/>
-    <axis xyz="0 1 0"/>
-    <dynamics damping="0.001" friction="0.001"/>
   </joint>
   <!-- ========== RPLIDAR A1 ========== -->
@@ -235,5 +235,4 @@
       <material name="CameraDark"/>
     </visual>
-    <!-- 镜头 -->
     <visual>
       <origin xyz="0.045 0.008 0.008" rpy="0 0 0"/>
@@ -270,5 +269,4 @@
     <origin xyz="0 0 0" rpy="0 0 0"/>
   </joint>
-  <!-- Gazebo 插件配置 -->
-  <xacro:include filename="$(find genbot_description)/urdf/genbot.gazebo.xacro" />
+  <xacro:include filename="$(find genbot_description)/urdf/genbot.gazebo.xacro"/>
 </robot>
